Commit message: removed useless rotations

File: iiwa_tool_description/urdf/iiwa_tool.urdf.xacro (robot description, xacro)
@@ -68,5 +68,5 @@
     <parent link="tool_link" />
     <child link = "tool_link_ee" />
-   <origin xyz="${tool_link_offset}" rpy="0 -${PI/2.0} 0" />
+   <origin xyz="${tool_link_offset}" rpy="0 0 0" />
   </joint>
 <!--  The TCP frame is here defined -->
@@ -78,5 +78,5 @@
     <parent link="tool_link" />
     <child link = "tool_link_ee_kuka" />
-    <origin xyz="${tool_link_offset}" rpy="0 ${PI} 0" />
+    <origin xyz="${tool_link_offset}" rpy="0 0 0" />
   </joint>
   <link name="tool_link_ee_kuka"/>

Commit message: actually, one rotation was needed

File: iiwa_tool_description/urdf/iiwa_tool.urdf.xacro (robot description, xacro)
@@ -68,5 +68,5 @@
     <parent link="tool_link" />
     <child link = "tool_link_ee" />
-   <origin xyz="${tool_link_offset}" rpy="0 0 0" />
+   <origin xyz="${tool_link_offset}" rpy="0 ${-PI/2.0} 0" />
   </joint>
 <!--  The TCP frame is here defined -->

Commit message: aligned

File: iiwa_tool_description/urdf/iiwa_tool.urdf.xacro (robot description, xacro)
@@ -6,10 +6,10 @@
   <!--Import the iiwa7 macro -->
   <xacro:include filename="$(find iiwa_description)/urdf/iiwa7.xacro"/>
-<!--  Define the origin of your 3D space
-      Here we define a box lying at 0,0,0 with some dimensions, in reality our robot is place on top of a metal cart with those dimensions.
-      This will include the cart in the scene and avoid the robot to hit it when using MoveIt!
-      If you don't want to have that you can define a basic world link (see commented lines)
+  <!--  Define the origin of your 3D space
+  Here we define a box lying at 0,0,0 with some dimensions, in reality our robot is place on top of a metal cart with those dimensions.
+  This will include the cart in the scene and avoid the robot to hit it when using MoveIt!
+  If you don't want to have that you can define a basic world link (see commented lines)
   -->
-<!--     <link name="world"/> -->
+  <!--     <link name="world"/> -->
   <link name="world">
     <visual>
@@ -29,5 +29,5 @@
     <static>true</static>
   </gazebo>
-<!-- Here we insert an iiwa7 robot in the scene, it's origin is just on top of the box previously defined. You can use 0,0,0 if you don't have that. -->
+  <!-- Here we insert an iiwa7 robot in the scene, it's origin is just on top of the box previously defined. You can use 0,0,0 if you don't have that. -->
   <xacro:iiwa7 hardware_interface="$(arg hardware_interface)" robot_name="$(arg robot_name)" parent="world">
     <origin xyz="0 0 0.84" rpy="0 0 0"/>
@@ -37,6 +37,6 @@
   <property name="tool_joint_offset" value="0.00 0.00 0.00" />
   <property name="tool_link_offset" value="0.00 0.00 0.1275" />
-<!--  Here we define a dummy joint between the tip of the iiwa7 and the base of the tool.
-      There is no offset between the two, that means the tool is attached at the robot flange. -->
+  <!--  Here we define a dummy joint between the tip of the iiwa7 and the base of the tool.
+  There is no offset between the two, that means the tool is attached at the robot flange. -->
   <joint name="tool_joint" type="fixed">
     <parent link="iiwa_link_ee" />
@@ -44,5 +44,5 @@
     <origin xyz="${tool_joint_offset}" rpy="0 ${PI/2.0} 0" />
   </joint>
-<!-- Here we define the geometry of the tool. We designed the tool ourselves, so we have a mesh file that represents it.
+  <!-- Here we define the geometry of the tool. We designed the tool ourselves, so we have a mesh file that represents it.
   Else, one can define it using a geometric representation that approximate it, like a cylinder (see commented lines) -->
   <link name="tool_link">
@@ -51,5 +51,5 @@
       <geometry>
 	<mesh filename="package://iiwa_tool_description/meshes/visual/tool.stl"/>
-<!-- 	<cylinder length="0.1275" radius="0.020"/> -->
+	<!-- 	<cylinder length="0.1275" radius="0.020"/> -->
       </geometry>
       <material name="Grey"/>
@@ -59,21 +59,21 @@
       <geometry>
 	<mesh filename="package://iiwa_tool_description/meshes/visual/tool.stl"/>
-<!-- 	<cylinder length="0.1275" radius="0.020"/> -->
+	<!-- 	<cylinder length="0.1275" radius="0.020"/> -->
       </geometry>
       <material name="Grey"/>
     </collision>
   </link>
-<!--  Here we define another dummy joint. It is placed at the end of the tool, so we can then attach a frame at its TCP for control -->
+  <!--  Here we define another dummy joint. It is placed at the end of the tool, so we can then attach a frame at its TCP for control -->
   <joint name="tool_tip_joint" type="fixed">
     <parent link="tool_link" />
     <child link = "tool_link_ee" />
-   <origin xyz="${tool_link_offset}" rpy="0 ${-PI/2.0} 0" />
+    <origin xyz="${tool_link_offset}" rpy="0 ${-PI/2.0} 0" />
   </joint>
-<!--  The TCP frame is here defined -->
+  <!--  The TCP frame is here defined -->
   <link name="tool_link_ee"/>
-<!-- Here we do the same as before, the resulting frame will be in the same position of the last one,
+  <!-- Here we do the same as before, the resulting frame will be in the same position of the last one,
   but we add a rotation to be aligned with the convention used by KUKA. So this fame will have exactly the same representation of the frame
   attached to this tool as defined in Sunrise Workbench! This is really useful when directly controlling the robot without MoveIt! -->
-    <joint name="tool_tip_joint_kuka" type="fixed">
+  <joint name="tool_tip_joint_kuka" type="fixed">
     <parent link="tool_link" />
     <child link = "tool_link_ee_kuka" />
