Commit message: updated moveit example

File: iiwa_tool/iiwa_tool_description/urdf/iiwa_tool.urdf.xacro (robot description, xacro)
@@ -71,16 +71,7 @@
     <parent link="tool_link" />
     <child link = "tool_link_ee" />
-    <origin xyz="${tool_link_offset}" rpy="0 ${-PI/2.0} 0" />
+    <origin xyz="${tool_link_offset}" rpy="0 0 0" />
   </joint>
   <!--  The TCP frame is here defined -->
   <link name="tool_link_ee"/>
-  <!-- Here we do the same as before, the resulting frame will be in the same position of the last one,
-  but we add a rotation to be aligned with the convention used by KUKA. So this fame will have exactly the same representation of the frame
-  attached to this tool as defined in Sunrise Workbench! This is really useful when directly controlling the robot without MoveIt! -->
-  <joint name="tool_tip_joint_kuka" type="fixed">
-    <parent link="tool_link" />
-    <child link = "tool_link_ee_kuka" />
-    <origin xyz="${tool_link_offset}" rpy="0 0 0" />
-  </joint>
-  <link name="tool_link_ee_kuka"/>
 </robot>

Commit message: fix tool orientation

File: iiwa_tool/iiwa_tool_description/urdf/iiwa_tool.urdf.xacro (robot description, xacro)
@@ -45,5 +45,5 @@
     <parent link="iiwa_link_ee" />
     <child link = "tool_link" />
-    <origin xyz="${tool_joint_offset}" rpy="0 ${PI/2.0} 0" />
+    <origin xyz="${tool_joint_offset}" rpy="0 0 0" />
   </joint>
   <!-- Here we define the geometry of the tool. We designed the tool ourselves, so we have a mesh file that represents it.
